File: PCB/OPEN_SPECTRO_PI_HAT.brd (EAGLE design)
At the start: 66 x 44 mm, 34 parts, among them IC1 DS3231/SO, J2 632722100213, J5 RASPBERRYPI-40-PIN-GPIO_PTH_N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

Commit message: Add files via upload
Connections:
- net GND: now also D3.A
Changed lines of the file:
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@@
 <via x="45" y="30.8" extent="1-16" drill="0.35" alwaysstop="yes">
 </via>
+<contactref element="D3" pad="A"/>
 </signal>
 <signal name="3.3V">
