File: PCB/OPEN_SPECTRO_PI_HAT.sch (EAGLE design)
At the start: 34 parts, among them IC1 DS3231/SO, J2 632722100213, J5 RASPBERRYPI-40-PIN-GPIO_PTH_N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

Commit message: Add files via upload
Connections:
- net GND: now also D3.C1
Changed lines of the file:
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@@
 <part name="GND14" library="_L_Symbols" library_urn="urn:adsk.wipprod:fs.file:vf.5DBbLlRNS2mpwKCAG8bHJA" deviceset="GND" device=""/>
 <part name="FR1" library="_L_Symbols" library_urn="urn:adsk.wipprod:fs.file:vf.5DBbLlRNS2mpwKCAG8bHJA" deviceset="SCH-FRAME-BIG" device=""/>
+<part name="GND18" library="_L_Symbols" library_urn="urn:adsk.wipprod:fs.file:vf.5DBbLlRNS2mpwKCAG8bHJA" deviceset="GND" device=""/>
 </parts>
 <sheets>
@@
 <attribute name="SHEET" x="373.38" y="5.08" size="1.778" layer="94" font="vector" ratio="10"/>
 <attribute name="LAST_DATE_TIME" x="313.69" y="5.08" size="1.778" layer="94" ratio="10"/>
+</instance>
+<instance part="GND18" gate="1" x="68.58" y="182.88" smashed="yes">
+<attribute name="VALUE" x="68.58" y="181.356" size="1.27" layer="96" font="vector" align="top-center"/>
 </instance>
 </instances>
@@
 <pinref part="GND14" gate="1" pin="BGND"/>
 </segment>
+<segment>
+<wire x1="68.58" y1="193.04" x2="68.58" y2="185.42" width="0.1524" layer="91"/>
+<pinref part="GND18" gate="1" pin="BGND"/>
+<pinref part="D3" gate="G$1" pin="C1"/>
+</segment>
 </net>
